Commit message: finished robot urdf ; note that we have a lot of unfinished/irrelevant files

File: ros2_ws/src/basic_robot_control/urdf/vehicle_blue.urdf (robot description, URDF)
Before this commit: robot vehicle_blue, 4 links, 3 joints
Links:
- added link base_link
Joints:
- added joint base_joint: type fixed, parent base_link, child chassis, origin xyz=0 0 0 rpy=0 0 0
